Commit message: add gazebo controls

File: description/robot.urdf.xacro (robot description, xacro)
@@ -2,3 +2,5 @@
 <robot xmlns:xacro="http://www.ros.org/wiki/xacro"  name="robot">
     <xacro:include filename="robot_base.xacro" />
+"
+    <xacro:include filename="gazebo_control.xacro" />
 </robot>

File: description/robot_base.xacro (robot description, xacro)
@@ -58,4 +58,7 @@
         </xacro:inertial_hollow_frame>
     </link>
+    <gazebo reference="chassis">
+        <material>Gazebo/White</material>
+    </gazebo>
                                                     <!-- RIGHT WHEEL LINK -->
     <joint name="right_wheel_joint" type="continuous">
@@ -82,4 +85,7 @@
         </xacro:inertial_cylinder>
     </link>
+    <gazebo reference="right_wheel">
+        <material>Gazebo/Orange</material>
+    </gazebo>
                                                     <!-- LEFT WHEEL LINK -->
     <joint name="left_wheel_joint" type="continuous">
@@ -106,4 +112,7 @@
         </xacro:inertial_cylinder>
     </link>
+    <gazebo reference="left_wheel">
+        <material>Gazebo/Orange</material>
+    </gazebo>
                                                     <!-- CASTER WHEEL LINKS -->
     <!--
@@ -136,4 +145,9 @@
         </xacro:inertial_sphere>
     </link>
+    <gazebo reference="caster_wheel_1">
+        <material>Gazebo/Blue</material>
+        <mu1 value="0.001"/>
+        <mu2 value="0.001"/>
+    </gazebo>
             <!-- Caster wheel 2 -->
     <joint name="caster_wheel_2_joint" type="fixed">
@@ -159,4 +173,9 @@
         </xacro:inertial_sphere>
     </link>
+    <gazebo reference="caster_wheel_2">
+        <material>Gazebo/Blue</material>
+        <mu1 value="0.001"/>
+        <mu2 value="0.001"/>
+    </gazebo>
         <!-- Caster wheel 3 -->
     <joint name="caster_wheel_3_joint" type="fixed">
@@ -182,4 +201,9 @@
         </xacro:inertial_sphere>
     </link>
+    <gazebo reference="caster_wheel_3">
+        <material>Gazebo/Blue</material>
+        <mu1 value="0.001"/>
+        <mu2 value="0.001"/>
+    </gazebo>
         <!-- Caster wheel 4 -->
     <joint name="caster_wheel_4_joint" type="fixed">
@@ -205,3 +229,8 @@
         </xacro:inertial_sphere>
     </link>
+    <gazebo reference="caster_wheel_4">
+        <material>Gazebo/Blue</material>
+        <mu1 value="0.001"/>
+        <mu2 value="0.001"/>
+    </gazebo>
 </robot>

Commit message: Add lidar simulation

File: description/robot.urdf.xacro (robot description, xacro)
@@ -2,5 +2,5 @@
 <robot xmlns:xacro="http://www.ros.org/wiki/xacro"  name="robot">
     <xacro:include filename="robot_base.xacro" />
-"
     <xacro:include filename="gazebo_control.xacro" />
+    <xacro:include filename="lidar.xacro"/>
 </robot>

File: description/robot_materials.xacro (robot description, xacro)
@@ -13,3 +13,6 @@
         <color rgba="0 0 0 1"/>
     </material>
+    <material name="red">
+        <color rgba="1 0 0 1"/>
+    </material>
 </robot>
