Commit message: finish basic visual model

File: description/robot_base.xacro (robot description, xacro)
@@ -2,23 +2,50 @@
 <robot xmlns:xacro="http://www.ros.org/wiki/xacro" >
     <xacro:include filename="robot_materials.xacro" />
-    <!-- BASE LINK -->
+                                                    <!-- BASE LINK -->
     <link name="base_link">
     </link>
-    <!-- CHASSIS LINK -->
+                                                    <!-- CHASSIS LINK -->
+    <!-- dimensiuni sasiu: 780x600mm
+        dimensiune profil: 40x40mm
+        L profil: 700mm
+        l profil: 600mm
+        Distanta mijloc sasiu - centru roti: 43.5mm
+    -->
     <joint name="chassis_joint" type="fixed">
         <parent link="base_link"/>
         <child link="chassis"/>
-        <origin xyz="-0.1 0 0"/>
+        <origin xyz="-0.39 0 0.0435"/>
     </joint>
     <link name="chassis">
-        <visual>
-            <origin xyz="0.39 0 0.075"/>
+        <visual> <!-- Back Profile -->
+            <origin xyz="0.02 0 0"/>
             <geometry>
-                <box size="0.78 0.6 0.15"/>
+                <box size="0.04 0.6 0.04"/>
             </geometry>
             <material name="white"/>
         </visual>
+        <visual> <!-- Front Profile -->
+            <origin xyz="0.76 0 0"/>
+            <geometry>
+                <box size="0.04 0.6 0.04"/>
+            </geometry>
+            <material name="white"/>
+        </visual>
+        <visual> <!-- Right Profile -->
+            <origin xyz="0.39 0.28 0"/>
+            <geometry>
+                <box size="0.7 0.04 0.04"/>
+            </geometry>
+            <material name="black"/>
+        </visual>
+        <visual> <!-- Left Profile -->
+            <origin xyz="0.39 -0.28 0"/>
+            <geometry>
+                <box size="0.7 0.04 0.04"/>
+            </geometry>
+            <material name="black"/>
+        </visual>
     </link>
-    <!-- RIGHT WHEEL LINK -->
+                                                    <!-- RIGHT WHEEL LINK -->
     <joint name="right_wheel_joint" type="continuous">
         <parent link="base_link"/>
@@ -30,10 +57,10 @@
         <visual>
             <geometry>
-                <cylinder radius="0.1" length="0.04"/>
+                <cylinder radius="0.05" length="0.04"/>
             </geometry>
             <material name="orange"/>
         </visual>
     </link>
-    <!-- LEFT WHEEL LINK -->
+                                                    <!-- LEFT WHEEL LINK -->
     <joint name="left_wheel_joint" type="continuous">
         <parent link="base_link"/>
@@ -45,9 +72,71 @@
         <visual>
             <geometry>
-                <cylinder radius="0.1" length="0.04"/>
+                <cylinder radius="0.05" length="0.04"/>
             </geometry>
             <material name="orange"/>
         </visual>
     </link>
+                                                    <!-- CASTER WHEEL LINKS -->
+    <!--
+        distanta centru roata - profil superior: 77.75mm
+        distanta X si Y centru roata - margine profil: 94.75mm
+        distanta roti L: 590.50mm
+        distanta roti l: 410.50mm
+    -->
+        <!-- Caster wheel 1 -->
+    <joint name="caster_wheel_1_joint" type="fixed">
+        <parent link="chassis"/>
+        <child link="caster_wheel_1"/>
+        <origin xyz="0.09475 0.20525 -0.058875"/>
+    </joint>
+    <link name="caster_wheel_1">
+        <visual>
+            <geometry>
+                <sphere radius="0.03775"/>
+            </geometry>
+            <material name="black"/>
+        </visual>
+    </link>
+            <!-- Caster wheel 2 -->
+    <joint name="caster_wheel_2_joint" type="fixed">
+        <parent link="chassis"/>
+        <child link="caster_wheel_2"/>
+        <origin xyz="0.09475 -0.20525 -0.058875"/>
+    </joint>
+    <link name="caster_wheel_2">
+        <visual>
+            <geometry>
+                <sphere radius="0.03775"/>
+            </geometry>
+            <material name="black"/>
+        </visual>
+    </link>
+        <!-- Caster wheel 3 -->
+    <joint name="caster_wheel_3_joint" type="fixed">
+        <parent link="chassis"/>
+        <child link="caster_wheel_3"/>
+        <origin xyz="0.68525 0.20525 -0.058875"/>
+    </joint>
+    <link name="caster_wheel_3">
+        <visual>
+            <geometry>
+                <sphere radius="0.03775"/>
+            </geometry>
+            <material name="black"/>
+        </visual>
+    </link>
+        <!-- Caster wheel 4 -->
+    <joint name="caster_wheel_4_joint" type="fixed">
+        <parent link="chassis"/>
+        <child link="caster_wheel_4"/>
+        <origin xyz="0.68525 -0.20525 -0.058875"/>
+    </joint>
+    <link name="caster_wheel_4">
+        <visual>
+            <geometry>
+                <sphere radius="0.03775"/>
+            </geometry>
+            <material name="black"/>
+        </visual>
+    </link>
 </robot>
-<!-- sasiu 600, roti ext 463 => 232.5-20 212.5 => 0.2125 -->

Commit message: add collision

File: description/robot_base.xacro (robot description, xacro)
@@ -46,4 +46,10 @@
             <material name="black"/>
         </visual>
+        <collision> <!-- Colision -->
+            <origin xyz="0.39 0 0"/>
+            <geometry>
+                <box size="0.78 0.6 0.04"/>
+            </geometry>
+        </collision>
     </link>
                                                     <!-- RIGHT WHEEL LINK -->
@@ -61,4 +67,9 @@
             <material name="orange"/>
         </visual>
+        <collision>
+            <geometry>
+                <cylinder radius="0.05" length="0.04"/>
+            </geometry>
+        </collision>
     </link>
                                                     <!-- LEFT WHEEL LINK -->
@@ -76,4 +87,9 @@
             <material name="orange"/>
         </visual>
+        <collision>
+            <geometry>
+                <cylinder radius="0.05" length="0.04"/>
+            </geometry>
+        </collision>
     </link>
                                                     <!-- CASTER WHEEL LINKS -->
@@ -97,4 +113,10 @@
             <material name="black"/>
         </visual>
+        <collision>
+            <geometry>
+                <sphere radius="0.03775"/>
+            </geometry>
+            <material name="black"/>
+        </collision>
     </link>
             <!-- Caster wheel 2 -->
@@ -111,4 +133,10 @@
             <material name="black"/>
         </visual>
+        <collision>
+            <geometry>
+                <sphere radius="0.03775"/>
+            </geometry>
+            <material name="black"/>
+        </collision>
     </link>
         <!-- Caster wheel 3 -->
@@ -125,4 +153,10 @@
             <material name="black"/>
         </visual>
+        <collision>
+            <geometry>
+                <sphere radius="0.03775"/>
+            </geometry>
+            <material name="black"/>
+        </collision>
     </link>
         <!-- Caster wheel 4 -->
@@ -139,4 +173,10 @@
             <material name="black"/>
         </visual>
+        <collision>
+            <geometry>
+                <sphere radius="0.03775"/>
+            </geometry>
+            <material name="black"/>
+        </collision>
     </link>
 </robot>

Commit message: add inertia

File: description/robot_base.xacro (robot description, xacro)
@@ -2,4 +2,5 @@
 <robot xmlns:xacro="http://www.ros.org/wiki/xacro" >
     <xacro:include filename="robot_materials.xacro" />
+    <xacro:include filename="inertial_macros.xacro" />
                                                     <!-- BASE LINK -->
     <link name="base_link">
@@ -52,4 +53,8 @@
             </geometry>
         </collision>
+                    <!-- Inertia -->
+        <xacro:inertial_hollow_frame mass="3.224" x="0.78" y="0.6" z="0.04">
+            <origin xyz="0.39 0 0" rpy="0 0 0" />
+        </xacro:inertial_hollow_frame>
     </link>
                                                     <!-- RIGHT WHEEL LINK -->
@@ -72,4 +77,8 @@
             </geometry>
         </collision>
+                    <!-- Inertia -->
+        <xacro:inertial_cylinder mass="0.1" length="0.04" radius="0.05">
+            <origin xyz="0 0 0" rpy="0 0 0"/>
+        </xacro:inertial_cylinder>
     </link>
                                                     <!-- LEFT WHEEL LINK -->
@@ -92,4 +101,8 @@
             </geometry>
         </collision>
+                    <!-- Inertia -->
+        <xacro:inertial_cylinder mass="0.1" length="0.04" radius="0.05">
+            <origin xyz="0 0 0" rpy="0 0 0"/>
+        </xacro:inertial_cylinder>
     </link>
                                                     <!-- CASTER WHEEL LINKS -->
@@ -117,6 +130,9 @@
                 <sphere radius="0.03775"/>
             </geometry>
-            <material name="black"/>
-        </collision>
+        </collision>
+        <!-- Inertia -->
+        <xacro:inertial_sphere mass="0.1" radius="0.03775">
+            <origin xyz="0 0 0" rpy="0 0 0"/>
+        </xacro:inertial_sphere>
     </link>
             <!-- Caster wheel 2 -->
@@ -137,6 +153,9 @@
                 <sphere radius="0.03775"/>
             </geometry>
-            <material name="black"/>
-        </collision>
+        </collision>
+        <!-- Inertia -->
+        <xacro:inertial_sphere mass="0.1" radius="0.03775">
+            <origin xyz="0 0 0" rpy="0 0 0"/>
+        </xacro:inertial_sphere>
     </link>
         <!-- Caster wheel 3 -->
@@ -157,6 +176,9 @@
                 <sphere radius="0.03775"/>
             </geometry>
-            <material name="black"/>
-        </collision>
+        </collision>
+        <!-- Inertia -->
+        <xacro:inertial_sphere mass="0.1" radius="0.03775">
+            <origin xyz="0 0 0" rpy="0 0 0"/>
+        </xacro:inertial_sphere>
     </link>
         <!-- Caster wheel 4 -->
@@ -177,6 +199,9 @@
                 <sphere radius="0.03775"/>
             </geometry>
-            <material name="black"/>
-        </collision>
+        </collision>
+        <!-- Inertia -->
+        <xacro:inertial_sphere mass="0.1" radius="0.03775">
+            <origin xyz="0 0 0" rpy="0 0 0"/>
+        </xacro:inertial_sphere>
     </link>
 </robot>

Commit message: create gazebo world and rviz config

File: description/robot_base.xacro (robot description, xacro)
@@ -126,5 +126,5 @@
         <parent link="chassis"/>
         <child link="caster_wheel_1"/>
-        <origin xyz="0.09475 0.20525 -0.058875"/>
+        <origin xyz="0.09475 0.20525 -0.05"/>
     </joint>
     <link name="caster_wheel_1">
@@ -154,5 +154,5 @@
         <parent link="chassis"/>
         <child link="caster_wheel_2"/>
-        <origin xyz="0.09475 -0.20525 -0.058875"/>
+        <origin xyz="0.09475 -0.20525 -0.05"/>
     </joint>
     <link name="caster_wheel_2">
@@ -182,5 +182,5 @@
         <parent link="chassis"/>
         <child link="caster_wheel_3"/>
-        <origin xyz="0.68525 0.20525 -0.058875"/>
+        <origin xyz="0.68525 0.20525 -0.05"/>
     </joint>
     <link name="caster_wheel_3">
@@ -210,5 +210,5 @@
         <parent link="chassis"/>
         <child link="caster_wheel_4"/>
-        <origin xyz="0.68525 -0.20525 -0.058875"/>
+        <origin xyz="0.68525 -0.20525 -0.05"/>
     </joint>
     <link name="caster_wheel_4">

Commit message: change colision from cylinder to sphere for sim

File: description/robot_base.xacro (robot description, xacro)
@@ -77,5 +77,5 @@
         <collision>
             <geometry>
-                <cylinder radius="0.05" length="0.04"/>
+                <sphere radius="0.05"/>
             </geometry>
         </collision>
@@ -104,5 +104,5 @@
         <collision>
             <geometry>
-                <cylinder radius="0.05" length="0.04"/>
+                <sphere radius="0.05"/>
             </geometry>
         </collision>
